Commit message: fixed the srdf to support different prefixes

File: robots/fr3_duo/fr3_duo.srdf.xacro (robot description, xacro)
@@ -8,6 +8,7 @@
   <!-- Which end-effector would be mounted at the flange?" -->
   <xacro:arg name="ee_id" default="franka_hand" />
-  <!-- Arm prefixes for the duo setup-->
-  <xacro:property name="arm_prefixes" value="${['left','right']}" />
+  <!-- Arm prefixes of the robots -->
+  <xacro:arg name="arm_prefixes" default="['left','right']" />
+  <xacro:property name="arm_prefixes_list" value="${$(arg arm_prefixes)}" />
   <xacro:property name="number_of_robots" value = "2"/>
   <xacro:macro name="missing_self_arm_collisions" params="full_arm_prefix">

File: robots/fr3_duo/fr3_duo.urdf.xacro (robot description, xacro)
@@ -46,5 +46,5 @@
   <!-- Thread priority for the hardware interface -->
   <xacro:arg name="thread_priority" default="50" />
-  <!-- Arm prefixes of the robot -->
+  <!-- Arm prefixes of the robots -->
   <xacro:arg name="arm_prefixes" default="['left','right']" />
   <xacro:property name="arm_prefixes_list" value="${$(arg arm_prefixes)}" />
