Commit message: fix: adding tests for gazebo revealed bug in fr3_duo

File: robots/fr3_duo/fr3_duo.urdf.xacro (robot description, xacro)
@@ -60,5 +60,5 @@
       <origin xyz="$(arg xyz)" rpy="$(arg rpy)"/>
       <parent link="world"/>
-      <child link="${modified_prefix}$(arg robot_type)_link0"/>
+      <child link="${base_mount_str}"/>
     </joint>
   </xacro:if>
