Commit message: revert lidar changes

File: robots/fer/fer.urdf.xacro (robot description, xacro)
@@ -44,7 +44,7 @@
   <xacro:property name="prefix" value="$(arg arm_prefix)"/>
   <xacro:property name="modified_prefix" value="${prefix + '_' if prefix else ''}"/>
-  <!--Position offset with respect the world-->
+  <!--Position offset with respect to the world-->
   <xacro:arg name="xyz" default="0 0 0" />
-  <!--Rotation offset with respect the world-->
+  <!--Rotation offset with respect to the world-->
   <xacro:arg name="rpy" default="0 0 0" />
   <xacro:if value="$(arg gazebo)">

File: robots/fp3/fp3.urdf.xacro (robot description, xacro)
@@ -44,7 +44,7 @@
   <xacro:property name="prefix" value="$(arg arm_prefix)"/>
   <xacro:property name="modified_prefix" value="${prefix + '_' if prefix else ''}"/>
-  <!--Position offset with respect the world-->
+  <!--Position offset with respect to the world-->
   <xacro:arg name="xyz" default="0 0 0" />
-  <!--Rotation offset with respect the world-->
+  <!--Rotation offset with respect to the world-->
   <xacro:arg name="rpy" default="0 0 0" />
   <xacro:if value="$(arg gazebo)">

File: robots/fr3/fr3.urdf.xacro (robot description, xacro)
@@ -44,7 +44,7 @@
   <xacro:property name="prefix" value="$(arg arm_prefix)"/>
   <xacro:property name="modified_prefix" value="${prefix + '_' if prefix else ''}"/>
-  <!--Position offset with respect the world-->
+  <!--Position offset with respect to the world-->
   <xacro:arg name="xyz" default="0 0 0" />
-  <!--Rotation offset with respect the world-->
+  <!--Rotation offset with respect to the world-->
   <xacro:arg name="rpy" default="0 0 0" />
   <xacro:if value="$(arg gazebo)">

File: robots/fr3v2/fr3v2.urdf.xacro (robot description, xacro)
@@ -44,7 +44,7 @@
   <xacro:property name="prefix" value="$(arg arm_prefix)"/>
   <xacro:property name="modified_prefix" value="${prefix + '_' if prefix else ''}"/>
-  <!--Position offset with respect the world-->
+  <!--Position offset with respect to the world-->
   <xacro:arg name="xyz" default="0 0 0" />
-  <!--Rotation offset with respect the world-->
+  <!--Rotation offset with respect to the world-->
   <xacro:arg name="rpy" default="0 0 0" />
   <xacro:if value="$(arg gazebo)">

File: robots/fr3v2_1/fr3v2_1.urdf.xacro (robot description, xacro)
@@ -44,7 +44,7 @@
   <xacro:property name="prefix" value="$(arg arm_prefix)"/>
   <xacro:property name="modified_prefix" value="${prefix + '_' if prefix else ''}"/>
-  <!--Position offset with respect the world-->
+  <!--Position offset with respect to the world-->
   <xacro:arg name="xyz" default="0 0 0" />
-  <!--Rotation offset with respect the world-->
+  <!--Rotation offset with respect to the world-->
   <xacro:arg name="rpy" default="0 0 0" />
   <xacro:if value="$(arg gazebo)">

File: robots/mobile_fr3_duo_v0_2/mobile_fr3_duo_v0_2.xacro (robot description, xacro)
@@ -32,5 +32,5 @@
     </xacro:if>
     <xacro:unless value="${gazebo}">
-         <xacro:property name="ros_control_flag_for_real_hardware" value ="true"/>
+         <xacro:property name="ros_control_flag_for_real_hardware" value ="${ros2_control}"/>
     </xacro:unless>
     <xacro:property name="number_of_robots" value = "3"/>

File: robots/tmrv0_2/tmrv0_2.ros2_control.xacro (robot description, xacro)
@@ -127,5 +127,5 @@
         </plugin>
       </gazebo>
-    </xacro:if>y
+    </xacro:if>
   </xacro:macro>
 </robot>

File: robots/tmrv0_2/tmrv0_2.xacro (robot description, xacro)
@@ -128,5 +128,5 @@
       <parent link="base_link" />
       <child link="lidar_front_mounting_point" />
-      <origin xyz="0.3275 0.2175 0.19065" rpy="0 0 ${pi/4}" />
+      <origin xyz="0.3275 0.2175 0.19065" rpy="0 ${pi} ${pi*3/4}" />
     </joint>
     <link name="lidar_rear_mounting_point"/>
@@ -134,5 +134,5 @@
       <parent link="base_link" />
       <child link="lidar_rear_mounting_point" />
-      <origin xyz="-0.3275 -0.2175 0.19065" rpy="0 0 ${pi*5/4}" />
+      <origin xyz="-0.3275 -0.2175 0.19065" rpy="0 ${pi} ${pi*7/4}" />
     </joint>
     <xacro:if value="${ros2_control}">
