Commit message: feat: head description added

File: robots/mobile_fr3_duo_v0_2/mobile_fr3_duo.ros2_control.xacro (robot description, xacro)
@@ -24,4 +24,5 @@
             is_async:=false
             thread_priority:=50
+            hand
             gazebo
             gazebo_effort
@@ -46,5 +47,5 @@
         </xacro:if>
         <xacro:if value="${use_fake_hardware == 0 and gazebo == 0}">
-          <!-- For real hardware, perhaps combine, but for now, assume gazebo -->
+          <!-- For real hardware but for now, assume gazebo always-->
         </xacro:if>
       </hardware>
@@ -181,4 +182,8 @@
       <xacro:general_purpose_io prefix="${arm2_prefix}_wy" command_interface="cartesian_velocity" index="4"/>
       <xacro:general_purpose_io prefix="${arm2_prefix}_wz" command_interface="cartesian_velocity" index="5"/>
+      <xacro:if value="${gazebo and hand}">
+        <xacro:configure_arm_joint joint_name="${arm1_prefix}_${arm1_type}_finger_joint1" initial_position="0.0" gazebo="${gazebo}" gazebo_effort="${gazebo_effort}"/>
+        <xacro:configure_arm_joint joint_name="${arm2_prefix}_${arm2_type}_finger_joint1" initial_position="0.0" gazebo="${gazebo}" gazebo_effort="${gazebo_effort}"/>
+      </xacro:if>
     </ros2_control>
     <xacro:if value="${gazebo}">

File: robots/mobile_fr3_duo_v0_2/mobile_fr3_duo_v0_2.urdf.xacro (robot description, xacro)
@@ -50,5 +50,5 @@
     <link name="base"/>
     <joint name="base_joint" type="fixed">
-      <parent link="${fixed_link_name}"/>
+      <parent link="base"/>
       <child link="base_link"/>
       <origin rpy="0 0 0" xyz="0 0 0"/>

File: robots/mobile_fr3_duo_v0_2/mobile_fr3_duo_v0_2.xacro (robot description, xacro)
@@ -27,4 +27,11 @@
     <xacro:include filename="$(find franka_description)/robots/tmrv0_2/tmrv0_2.xacro"/>
     <xacro:include filename="$(find franka_description)/robots/mobile_fr3_duo_v0_2/mobile_fr3_duo.ros2_control.xacro"/>
+    <xacro:include filename="$(find franka_description)/robots/fr3_duo/fr3_duo_head.xacro" />
+    <xacro:if value="${gazebo}">
+        <xacro:property name="ros_control_flag_for_real_hardware" value ="false"/>
+    </xacro:if>
+    <xacro:unless value="${gazebo}">
+         <xacro:property name="ros_control_flag_for_real_hardware" value ="true"/>
+    </xacro:unless>
     <xacro:property name="number_of_robots" value = "3"/>
     <xacro:property name="arm_prefixes_list" value="${['','left','right']}" />
@@ -35,5 +42,5 @@
                 <xacro:tmrv0_2 mobile_robot_type="${robot_type_i}"
                     robot_ip="${robot_ips_list[i]}"
-                    ros2_control="false"
+                    ros2_control="${ros_control_flag_for_real_hardware}"
                     use_fake_hardware="${use_fake_hardware}"
                     fake_sensor_commands="${fake_sensor_commands}"
@@ -90,4 +97,7 @@
                 <origin xyz="0 0 0" rpy="0 0 0" />
             </xacro:mount>
+            <xacro:head name="head" parent="mount_link">
+                <origin xyz="0 0 0.167" rpy="0 0 0" />
+            </xacro:head>
         </xacro:if>
         <xacro:unless value="${robot_type_i == 'tmrv0_2'}">
@@ -128,5 +138,5 @@
                                 safety_distance="${safety_distance}"
                                 with_sc="${with_sc}"
-                                ros2_control="false"
+                                ros2_control="${ros_control_flag_for_real_hardware}"
                                 robot_ip="${robot_ips_list[i]}"
                                 use_fake_hardware="${use_fake_hardware}"
@@ -145,13 +155,16 @@
     </xacro:macro>
     <xacro:loop i="0"/>
-    <xacro:mobile_fr3_duo_ros2_control mobile_robot_type="tmrv0_2"
-                                        robot_types="${robot_types_list}"
-                                        arm_prefixes="${arm_prefixes_list}"
-                                        robot_ips="${robot_ips_list}"
-                                        use_fake_hardware="$(arg use_fake_hardware)"
-                                        fake_sensor_commands="$(arg fake_sensor_commands)"
-                                        gazebo="$(arg gazebo)"
-                                        gazebo_effort="$(arg gazebo_effort)"
-                                        robot_namespace=""/>
+    <xacro:if value="${gazebo}">
+        <xacro:mobile_fr3_duo_ros2_control mobile_robot_type="tmrv0_2"
+                                            robot_types="${robot_types_list}"
+                                            arm_prefixes="${arm_prefixes_list}"
+                                            robot_ips="${robot_ips_list}"
+                                            hand="${hand}"
+                                            use_fake_hardware="${use_fake_hardware}"
+                                            fake_sensor_commands="${fake_sensor_commands}"
+                                            gazebo="${gazebo}"
+                                            gazebo_effort="${gazebo_effort}"
+                                            robot_namespace=""/>
+    </xacro:if>
   </xacro:macro>
 </robot>

Commit message: fix: mfr3duo arm_prefixes index

File: robots/mobile_fr3_duo_v0_2/mobile_fr3_duo.ros2_control.xacro (robot description, xacro)
@@ -83,6 +83,6 @@
       <xacro:property name="arm1_type" value="${robot_types_list[1]}"/>
       <xacro:property name="arm2_type" value="${robot_types_list[2]}"/>
-      <xacro:property name="arm1_prefix" value="${arm_prefixes_list[1]}"/>
-      <xacro:property name="arm2_prefix" value="${arm_prefixes_list[2]}"/>
+      <xacro:property name="arm1_prefix" value="${arm_prefixes_list[0]}"/>
+      <xacro:property name="arm2_prefix" value="${arm_prefixes_list[1]}"/>
       <!-- Left arm -->
       <xacro:configure_arm_joint joint_name="${arm1_prefix}_${arm1_type}_joint1" initial_position="0.0"
